Commit message: enable multiple quads support

File: crazyflie_gazebo/models/rotors_description/urdf/component_snippets.xacro (robot description, xacro)
@@ -223,8 +223,4 @@
         <noiseUniformLinearVelocity>${noise_uniform_linear_velocity}</noiseUniformLinearVelocity> <!-- symmetric bounds of uniform noise [m/s] -->
         <noiseUniformAngularVelocity>${noise_uniform_angular_velocity}</noiseUniformAngularVelocity> <!-- symmetric bounds of uniform noise [rad/s] -->
-        <xacro:if value="${enable_odometry_map}">
-          <covarianceImage>package://rotors_gazebo/resource/${odometry_map}</covarianceImage> <!-- a bitmap image describing where the sensor works (white), and where not (black) -->
-          <covarianceImageScale>${image_scale}</covarianceImageScale> <!-- the scale of the image in the gazebo world, if set to 1.0, 1 pixel in the image corresponds to 1 meter in the world -->
-        </xacro:if>
       </plugin>
     </gazebo>

File: crazyflie_gazebo/models/rotors_description/urdf/multirotor_base.xacro (robot description, xacro)
@@ -38,5 +38,5 @@
         <origin xyz="0 0 0" rpy="0 0 0" />
         <geometry>
-          <mesh filename="package://rotors_description/meshes/${mesh_file}"
+          <mesh filename="$(arg rotors_description_dir)/meshes/${mesh_file}"
             scale="${mesh_scale}" />
           <!-- <box size="${body_width} ${body_width} ${body_height}"/> --> <!-- [m] [m] [m] -->
@@ -98,9 +98,9 @@
           <!-- <mesh filename="package://rotors_description/meshes/propeller_${direction}.dae" -->
           <xacro:if value="${use_own_mesh}">
-            <mesh filename="package://rotors_description/meshes/${mesh}"
+            <mesh filename="$(arg rotors_description_dir)/meshes/${mesh}"
               scale="${mesh_scale}" />
           </xacro:if>
           <xacro:unless value="${use_own_mesh}">
-            <mesh filename="package://rotors_description/meshes/${mesh}_${direction}.dae" scale="${mesh_scale}" />
+            <mesh filename="$(arg rotors_description_dir)/meshes/${mesh}_${direction}.dae" scale="${mesh_scale}" />
           </xacro:unless>
           <!-- <box size="${2*radius_rotor} 0.01 0.005"/> -->

Commit message: generalized topics name + update worlds params

File: crazyflie_gazebo/models/rotors_description/urdf/component_snippets.xacro (robot description, xacro)
@@ -20,4 +20,9 @@
 -->
 <robot xmlns:xacro="http://ros.org/wiki/xacro">
+  <!-- Global variables -->
+  <xacro:property name='imu_topic' value='gazebo/imu' />
+  <xacro:property name='mag_topic' value='gazebo/magnetic_field' />
+  <xacro:property name='pressure_topic' value='gazebo/air_pressure' />
+  <xacro:property name="motorsSpeedTopic" value="/gazebo/command/motor_speed"/>
   <!-- Macro to add logging to a bag file. -->
   <xacro:macro name="bag_plugin_macro"
@@ -59,5 +64,5 @@
   <!-- Macro to add an IMU. -->
   <xacro:macro name="imu_plugin_macro"
-    params="namespace imu_suffix parent_link imu_topic
+    params="namespace imu_suffix parent_link imu_topic rate
       mass_imu_sensor gyroscope_noise_density gyroscope_random_walk
       gyroscope_bias_correlation_time gyroscope_turn_on_bias_sigma
@@ -87,4 +92,5 @@
         <linkName>${namespace}/imu${imu_suffix}_link</linkName> <!-- (string, required): name of the body which holds the IMU sensor -->
         <imuTopic>${imu_topic}</imuTopic> <!-- (string): name of the sensor output topic and prefix of service names (defaults to imu) -->
+        <rate>${rate}</rate> <!-- Imu frequency update in Hz -->
         <gyroscopeNoiseDensity>${gyroscope_noise_density}</gyroscopeNoiseDensity> <!-- Gyroscope noise density (two-sided spectrum) [rad/s/sqrt(Hz)] -->
         <gyroscopeRandomWalk>${gyroscope_random_walk}</gyroscopeRandomWalk> <!-- Gyroscope bias random walk [rad/s/s/sqrt(Hz)] -->

File: crazyflie_gazebo/models/rotors_description/urdf/crazyflie_base.xacro (robot description, xacro)
@@ -28,7 +28,4 @@
   <xacro:property name="enable_parameters" value="$(arg enable_parameters)" />
   <xacro:property name="enable_ground_truth" value="$(arg enable_ground_truth)" />
-  <xacro:property name='imu_topic' value='gazebo/imu' />
-  <xacro:property name='mag_topic' value='gazebo/magnetic_field' />
-  <xacro:property name='pressure_topic' value='gazebo/air_pressure' />
   <xacro:include filename="$(arg rotors_description_dir)/urdf/component_snippets.xacro"/>
   <!-- Instantiate crazyflie "mechanics" -->
@@ -54,4 +51,5 @@
     imu_topic="${imu_topic}"
     mass_imu_sensor="0.00001"
+    rate="500"
     gyroscope_noise_density="1.7667e-4"
     gyroscope_random_walk="9.2542e-06"
@@ -70,4 +68,5 @@
       parent_link="base_link"
       imu_topic="${imu_topic}"
+      rate="400"
       mass_imu_sensor="0.00001"
       gyroscope_noise_density="0.0"
@@ -116,24 +115,26 @@
     rate="100">
   </xacro:lps_plugin_macro>
-  <xacro:crtp_interface_macro
-    namespace="${namespace}"
-    imu_sub_topic="${imu_topic}"
-    mag_sub_topic="${mag_topic}"
-    pressure_sub_topic="${pressure_topic}"
-    motors_speeds_pub_topic="gazebo/command/motor_speed"
-    rotor_count="4"
-    uri="${uri}"
-    roll_trim="${roll_trim}"
-    pitch_trim="${pitch_trim}"
-    enable_logging="${enable_logging}"
-    use_ros_time="${use_ros_time}"
-    enable_logging_imu="${enable_logging_imu}"
-    enable_logging_magnetic_field="${enable_logging_magnetic_field}"
-    enable_logging_temperature="${enable_logging_temperature}"
-    enable_logging_pressure="${enable_logging_pressure}"
-    enable_logging_battery="${enable_logging_battery}"
-    enable_logging_packets="${enable_logging_packets}"
-    enable_parameters="${enable_parameters}">
-  </xacro:crtp_interface_macro>
+  <xacro:if value="$(arg is_hitl)">
+    <xacro:crtp_interface_macro
+      namespace="${namespace}"
+      imu_sub_topic="${imu_topic}"
+      mag_sub_topic="${mag_topic}"
+      pressure_sub_topic="${pressure_topic}"
+      motors_speeds_pub_topic="${motorsSpeedTopic}"
+      rotor_count="4"
+      uri="${uri}"
+      roll_trim="${roll_trim}"
+      pitch_trim="${pitch_trim}"
+      enable_logging="${enable_logging}"
+      use_ros_time="${use_ros_time}"
+      enable_logging_imu="${enable_logging_imu}"
+      enable_logging_magnetic_field="${enable_logging_magnetic_field}"
+      enable_logging_temperature="${enable_logging_temperature}"
+      enable_logging_pressure="${enable_logging_pressure}"
+      enable_logging_battery="${enable_logging_battery}"
+      enable_logging_packets="${enable_logging_packets}"
+      enable_parameters="${enable_parameters}">
+    </xacro:crtp_interface_macro>
+  </xacro:if>
   <xacro:if value="${enable_ground_truth}">
     <!-- Odometry Sensor -->

File: crazyflie_gazebo/models/rotors_description/urdf/multirotor_base.xacro (robot description, xacro)
@@ -107,9 +107,9 @@
         </geometry>
       </visual>
-      <collision>
+      <!--<collision>
         <geometry>
-          <cylinder length="0.005" radius="${radius_rotor}" /> <!-- [m] -->
+          <cylinder length="0.005" radius="${radius_rotor}" />
         </geometry>
-      </collision>
+      </collision> -->
     </link>
     <gazebo>
@@ -124,5 +124,5 @@
         <motorConstant>${motor_constant}</motorConstant>
         <momentConstant>${moment_constant}</momentConstant>
-        <commandSubTopic>/gazebo/command/motor_speed</commandSubTopic>
+        <commandSubTopic>${motorsSpeedTopic}</commandSubTopic>
         <motorNumber>${motor_number}</motorNumber>
         <rotorDragCoefficient>${rotor_drag_coefficient}</rotorDragCoefficient>

Commit message: integrate real behavior into gazebo + new worlds + minor fixes

File: crazyflie_gazebo/models/rotors_description/urdf/component_snippets.xacro (robot description, xacro)
@@ -284,3 +284,11 @@
     </gazebo>
   </xacro:macro>
+  <xacro:macro name="ghost_plugin_macro"
+    params="poseTopic">
+    <gazebo>
+      <plugin name="cfGhost_plugin" filename="libgazebo_cfGhost_plugin.so">
+        <poseTopic>${poseTopic}</poseTopic>
+      </plugin>
+    </gazebo>
+  </xacro:macro>
 </robot>
