Commit message: clean up + minor fixes

File: crazyflie_gazebo/models/rotors_description/urdf/cfHandler_base.xacro (robot description, xacro)
@@ -18,4 +18,5 @@
   <xacro:property name="cfPrefix" value="$(arg cfPrefix)" />
   <xacro:property name="udpPort" value="$(arg udpPort)" />
+  <xacro:property name="firstIndex" value="$(arg firstIndex)" />
   <xacro:include filename="$(arg rotors_description_dir)/urdf/component_snippets.xacro"/>
   <link name="base_link"></link>
@@ -41,4 +42,5 @@
         <cfPrefix>${cfPrefix}</cfPrefix>
         <udpPort>${udpPort}</udpPort>
+        <firstIndex>${firstIndex}</firstIndex>
       </plugin>
   </gazebo>

Commit message: add hitl to cfHandler + simplify cf gazebo model

File: crazyflie_gazebo/models/rotors_description/urdf/cfHandler_base.xacro (robot description, xacro)
@@ -17,5 +17,5 @@
   <xacro:property name="nbQuads" value="$(arg nbQuads)" />
   <xacro:property name="cfPrefix" value="$(arg cfPrefix)" />
-  <xacro:property name="udpPort" value="$(arg udpPort)" />
+  <xacro:property name="uri" value="$(arg uri)" />
   <xacro:property name="firstIndex" value="$(arg firstIndex)" />
   <xacro:include filename="$(arg rotors_description_dir)/urdf/component_snippets.xacro"/>
@@ -41,5 +41,5 @@
         <nbQuads>${nbQuads}</nbQuads>
         <cfPrefix>${cfPrefix}</cfPrefix>
-        <udpPort>${udpPort}</udpPort>
+        <uri>${uri}</uri>
         <firstIndex>${firstIndex}</firstIndex>
       </plugin>

File: crazyflie_gazebo/models/rotors_description/urdf/component_snippets.xacro (robot description, xacro)
@@ -256,32 +256,4 @@
     </gazebo>
   </xacro:macro>
-  <!-- CRTP Interface -->
-  <xacro:macro name="crtp_interface_macro"
-    params="namespace imu_sub_topic mag_sub_topic pressure_sub_topic motors_speeds_pub_topic rotor_count uri roll_trim pitch_trim enable_logging use_ros_time enable_logging_imu enable_logging_magnetic_field enable_logging_temperature enable_logging_pressure enable_logging_battery enable_logging_packets enable_parameters">
-    <gazebo>
-      <plugin name="crtp_interface" filename="libgazebo_crtp_interface.so">
-        <robotNamespace>${namespace}</robotNamespace>
-        <imuSubTopic>${imu_sub_topic}</imuSubTopic>
-        <magnetometerTopic>${mag_sub_topic}</magnetometerTopic>
-        <pressureTopic>${pressure_sub_topic}</pressureTopic>
-        <motorSpeedsPubTopic>${motors_speeds_pub_topic}</motorSpeedsPubTopic>
-        <crazyflieURI>${uri}</crazyflieURI>
-        <rollTrim>${roll_trim}</rollTrim>
-        <pitchTrim>${pitch_trim}</pitchTrim>
-        <enableLogging>${enable_logging}</enableLogging>
-        <useRosTime>${use_ros_time}</useRosTime>
-        <enableLoggingImu>${enable_logging_imu}</enableLoggingImu>
-        <enableLoggingTemperature>${enable_logging_temperature}</enableLoggingTemperature>
-        <enableLoggingMagneticField>${enable_logging_magnetic_field}</enableLoggingMagneticField>
-        <enableLoggingPressure>${enable_logging_pressure}</enableLoggingPressure>
-        <enableLoggingBattery>${enable_logging_battery}</enableLoggingBattery>
-        <enableLoggingPackets>${enable_logging_packets}</enableLoggingPackets>
-        <enableParameters>${enable_parameters}</enableParameters>
-        <!-- <gpsUpdateFreq>${gps_update_freq}</gpsUpdateFreq> Frequency of HIL GPS messages [Hz] -->
-        <rotorCount>${rotor_count}</rotorCount>
-        <!-- https://www.ngdc.noaa.gov/geomag/WMM/calculators.shtml -->
-      </plugin>
-    </gazebo>
-  </xacro:macro>
   <xacro:macro name="ghost_plugin_macro"
     params="poseTopic">

File: crazyflie_gazebo/models/rotors_description/urdf/crazyflie_base.xacro (robot description, xacro)
@@ -11,20 +11,4 @@
   <xacro:arg name='enable_logging' default='false' />
   <xacro:arg name='log_file' default='crazyflie' />
-  <!-- crtp arguments -->
-<!--   <xacro:property name="uri" value="usb://0" /> -->
-<!--   <xacro:property name="uri" value="INADDR_ANY://19950" />
-  <xacro:property name='enable_ground_truth' value='true' /> -->
-  <xacro:property name="uri" value="$(arg uri)" />
-  <xacro:property name="roll_trim" value="$(arg roll_trim)" />
-  <xacro:property name="pitch_trim" value="$(arg pitch_trim)" />
-  <xacro:property name="enable_logging" value="$(arg enable_logging)" />
-  <xacro:property name="enable_logging_imu" value="$(arg enable_logging_imu)" />
-  <xacro:property name="enable_logging_temperature" value="$(arg enable_logging_temperature)" />
-  <xacro:property name="enable_logging_pressure" value="$(arg enable_logging_pressure)" />
-  <xacro:property name="enable_logging_battery" value="$(arg enable_logging_battery)" />
-  <xacro:property name="enable_logging_packets" value="$(arg enable_logging_packets)" />
-  <xacro:property name="enable_logging_magnetic_field" value="$(arg enable_logging_magnetic_field)" />
-  <xacro:property name="use_ros_time" value="$(arg use_ros_time)" />
-  <xacro:property name="enable_parameters" value="$(arg enable_parameters)" />
   <xacro:property name="enable_ground_truth" value="$(arg enable_ground_truth)" />
   <xacro:include filename="$(arg rotors_description_dir)/urdf/component_snippets.xacro"/>
@@ -115,26 +99,4 @@
     rate="100">
   </xacro:lps_plugin_macro>
-  <xacro:if value="$(arg is_hitl)">
-    <xacro:crtp_interface_macro
-      namespace="${namespace}"
-      imu_sub_topic="${imu_topic}"
-      mag_sub_topic="${mag_topic}"
-      pressure_sub_topic="${pressure_topic}"
-      motors_speeds_pub_topic="${motorsSpeedTopic}"
-      rotor_count="4"
-      uri="${uri}"
-      roll_trim="${roll_trim}"
-      pitch_trim="${pitch_trim}"
-      enable_logging="${enable_logging}"
-      use_ros_time="${use_ros_time}"
-      enable_logging_imu="${enable_logging_imu}"
-      enable_logging_magnetic_field="${enable_logging_magnetic_field}"
-      enable_logging_temperature="${enable_logging_temperature}"
-      enable_logging_pressure="${enable_logging_pressure}"
-      enable_logging_battery="${enable_logging_battery}"
-      enable_logging_packets="${enable_logging_packets}"
-      enable_parameters="${enable_parameters}">
-    </xacro:crtp_interface_macro>
-  </xacro:if>
   <xacro:if value="${enable_ground_truth}">
     <!-- Odometry Sensor -->
